File: Turret2_portable/mcu.kicad_sch (KiCad schematic)
At the start: 48 parts, among them IC2 SN74AHCT125PWR, J10 ROTATE_X, J2 TC2050-IDC, J3 GUN_LEFT, J4 GUN_RIGHT, J7 WING_LEFT, J8 WING_RIGHT, J9 ROTATE_Z, SW1 USB / JTAG, SW2 Prog, SW3 Reset, U6 LSM6DSOXTR, U7 ESP32-S3-MINI-1, U9 MAX98357A

Commit message: Portable KiCad copy: R18 100 ohm in the schematic, KiCad re-save
R18 (IO33 -> green LED D4) goes from 1 kohm to 100 ohm in mcu.kicad_sch,
as already documented on 19.10.2026. The rest of the diff is KiCad
reordering the schematic files on save. Adds the 2026-10-19 backup.

Co-Authored-By: Claude Opus 5.5 <noreply@anthropic.com>
Parts:
- R18: value 1K -> 100Ω
Changed lines of the file:
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@@
 			)
 		)
-		(property "Value" "1K"
+		(property "Value" "100Ω"
 			(at 128.27 69.85 90)
 			(show_name no)
